File: e73-breakout.kicad_sch (KiCad schematic)
At the start: 8 parts, among them J1 Conn_ARM_JTAG_SWD_10, J2 Pin, J3 Pin, J4 Pin, SW1 2x3mm, U1 E73-2G4M04S1D-51822

Commit message: Some updates and pictures.
Parts:
- C1: footprint Capacitor_SMD:C_0805_2012Metric_Pad1.18x1.45mm_HandSolder -> Capacitor_THT:C_Disc_D3.0mm_W1.6mm_P2.50mm
- J1: footprint Connector_PinHeader_1.27mm:PinHeader_2x05_P1.27mm_Vertical_SMD -> Connector_PinHeader_1.27mm:PinHeader_2x05_P1.27mm_Vertical
- R1: footprint Resistor_SMD:R_0603_1608Metric -> Resistor_THT:R_Axial_DIN0204_L3.6mm_D1.6mm_P5.08mm_Horizontal
- SW1: footprint Button_Switch_SMD:SW_Push_SPST_NO_Alps_SKRK -> kbd:ResetSW_1side
Connections:
- net SWO: no longer names the net of J1.6 (SWO/TDO)
- no-connect marks 1 -> 2
Changed lines of the file:
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@@
   (junction (at 63.5 157.48) (diameter 0) (color 0 0 0 0)
   )
+  (no_connect (at 76.2 144.78))
   (no_connect (at 76.2 147.32))
   (wire (pts (xy 53.34 101.6) (xy 57.15 101.6))
@@
   )
   (label "SWDCLK" (at 76.2 139.7 0) (fields_autoplaced)
-    (effects (font (size 1.27 1.27)) (justify left bottom))
-  )
-  (label "SWO" (at 76.2 144.78 0) (fields_autoplaced)
     (effects (font (size 1.27 1.27)) (justify left bottom))
   )
@@
       (effects (font (size 1.27 1.27)) (justify right))
     )
-    (property "Footprint" "Connector_PinHeader_1.27mm:PinHeader_2x05_P1.27mm_Vertical_SMD" (at 63.5 142.24 0)
+    (property "Footprint" "Connector_PinHeader_1.27mm:PinHeader_2x05_P1.27mm_Vertical" (at 63.5 142.24 0)
       (effects (font (size 1.27 1.27)) hide)
     )
@@
       (effects (font (size 1.27 1.27)) (justify left))
     )
-    (property "Footprint" "Capacitor_SMD:C_0805_2012Metric_Pad1.18x1.45mm_HandSolder" (at 102.5652 33.02 0)
+    (property "Footprint" "Capacitor_THT:C_Disc_D3.0mm_W1.6mm_P2.50mm" (at 102.5652 33.02 0)
       (effects (font (size 1.27 1.27)) hide)
     )
@@
       (effects (font (size 1.27 1.27)) (justify right))
     )
-    (property "Footprint" "Resistor_SMD:R_0603_1608Metric" (at 108.458 73.66 90)
+    (property "Footprint" "Resistor_THT:R_Axial_DIN0204_L3.6mm_D1.6mm_P5.08mm_Horizontal" (at 108.458 73.66 90)
       (effects (font (size 1.27 1.27)) hide)
     )
@@
       (effects (font (size 1.27 1.27)) hide)
     )
-    (property "Footprint" "Button_Switch_SMD:SW_Push_SPST_NO_Alps_SKRK" (at 115.316 72.39 0)
-      (effects (font (size 1.27 1.27)) hide)
-    )
+    (property "Footprint" "kbd:ResetSW_1side" (at 115.316 72.39 0)
+      (effects (font (size 1.27 1.27)) hide)
+    )
